File: pcb/lora_end_device/lora_end_device.sch (KiCad schematic (older format))
At the start: 31 parts, among them J1 USB_B_Micro, J2 UFL, J3 SMA, J4 UART, J5 Reset, J6 PRG, U1 TC1047A, U2 MCP6021, U3 LD1117, U4 RFM95W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

Commit message: asociacion huellas, posicionamiento, borde
Parts:
- removed U1: TC1047A, Package_TO_SOT_SMD:SOT-23, symbol Sensor_Temperature:TC1047AxNB
- added J7: Sensor, Connector_PinHeader_2.54mm:PinHeader_1x03_P2.54mm_Vertical, symbol Connector_Generic:Conn_01x03
Changed lines of the file:
@@
-$EndComp
-$Comp
-L Sensor_Temperature:TC1047AxNB U1
-U 1 1 60DF79A2
-P 2000 3900
-F 0 "U1" H 1650 4300 50  0000 R CNN
-F 1 "TC1047A" H 1900 4200 50  0000 R CNN
-F 2 "Package_TO_SOT_SMD:SOT-23" H 2000 3500 50  0001 C CNN
-F 3 "http://ww1.microchip.com/downloads/en/DeviceDoc/21498D.pdf" H 1850 4150 50  0001 C CNN
-	1    2000 3900
-	1    0    0    -1
 $EndComp
 $Comp
@@
 	2900 3900 2950 3900
 Connection ~ 4250 3800
-Wire Wire Line
-	2400 3900 2550 3900
-Wire Wire Line
-	2000 4200 2000 4400
 $Comp
 L power:+3.3V #PWR01
@@
 	1    0    0    -1
 $EndComp
-Wire Wire Line
-	2000 3600 2000 3400
 Wire Wire Line
 	2900 6100 3350 6100
@@
 	-1   0    0    -1
 $EndComp
+$Comp
+L Connector_Generic:Conn_01x03 J7
+U 1 1 610E4A12
+P 1800 3900
+F 0 "J7" H 1880 3942 50  0000 L CNN
+F 1 "Sensor" H 1880 3851 50  0000 L CNN
+F 2 "Connector_PinHeader_2.54mm:PinHeader_1x03_P2.54mm_Vertical" H 1800 3900 50  0001 C CNN
+F 3 "~" H 1800 3900 50  0001 C CNN
+	1    1800 3900
+	-1   0    0    1
+$EndComp
+Wire Wire Line
+	2000 3400 2000 3800
+Wire Wire Line
+	2000 3900 2550 3900
+Wire Wire Line
+	2000 4000 2000 4400
 $EndSCHEMATC

Commit message: reubicación de conector SMA
Parts:
- added FID1, FID2, FID3: Fiducial, Fiducial:Fiducial_0.75mm_Mask1.5mm, symbol Mechanical:Fiducial
- H1, H2, H3, H4: footprint MountingHole:MountingHole_3.2mm_M3 -> MountingHole:MountingHole_2.5mm_Pad
Changed lines of the file:
@@
 F 0 "H1" H 1600 1196 50  0000 L CNN
 F 1 "MountingHole" H 1600 1105 50  0000 L CNN
-F 2 "MountingHole:MountingHole_3.2mm_M3" H 1500 1150 50  0001 C CNN
+F 2 "MountingHole:MountingHole_2.5mm_Pad" H 1500 1150 50  0001 C CNN
 F 3 "~" H 1500 1150 50  0001 C CNN
 	1    1500 1150
@@
 F 0 "H3" H 2500 1196 50  0000 L CNN
 F 1 "MountingHole" H 2500 1105 50  0000 L CNN
-F 2 "MountingHole:MountingHole_3.2mm_M3" H 2400 1150 50  0001 C CNN
+F 2 "MountingHole:MountingHole_2.5mm_Pad" H 2400 1150 50  0001 C CNN
 F 3 "~" H 2400 1150 50  0001 C CNN
 	1    2400 1150
@@
 F 0 "H2" H 1600 1846 50  0000 L CNN
 F 1 "MountingHole" H 1600 1755 50  0000 L CNN
-F 2 "MountingHole:MountingHole_3.2mm_M3" H 1500 1800 50  0001 C CNN
+F 2 "MountingHole:MountingHole_2.5mm_Pad" H 1500 1800 50  0001 C CNN
 F 3 "~" H 1500 1800 50  0001 C CNN
 	1    1500 1800
@@
 F 0 "H4" H 2550 1846 50  0000 L CNN
 F 1 "MountingHole" H 2550 1755 50  0000 L CNN
-F 2 "MountingHole:MountingHole_3.2mm_M3" H 2450 1800 50  0001 C CNN
+F 2 "MountingHole:MountingHole_2.5mm_Pad" H 2450 1800 50  0001 C CNN
 F 3 "~" H 2450 1800 50  0001 C CNN
 	1    2450 1800
@@
 Wire Wire Line
 	2000 4000 2000 4400
+$Comp
+L Mechanical:Fiducial FID1
+U 1 1 61040CDB
+P 3350 1100
+F 0 "FID1" H 3435 1146 50  0000 L CNN
+F 1 "Fiducial" H 3435 1055 50  0000 L CNN
+F 2 "Fiducial:Fiducial_0.75mm_Mask1.5mm" H 3350 1100 50  0001 C CNN
+F 3 "~" H 3350 1100 50  0001 C CNN
+	1    3350 1100
+	1    0    0    -1
+$EndComp
+$Comp
+L Mechanical:Fiducial FID2
+U 1 1 610414A1
+P 3350 1500
+F 0 "FID2" H 3435 1546 50  0000 L CNN
+F 1 "Fiducial" H 3435 1455 50  0000 L CNN
+F 2 "Fiducial:Fiducial_0.75mm_Mask1.5mm" H 3350 1500 50  0001 C CNN
+F 3 "~" H 3350 1500 50  0001 C CNN
+	1    3350 1500
+	1    0    0    -1
+$EndComp
+$Comp
+L Mechanical:Fiducial FID3
+U 1 1 61041EF6
+P 3350 1900
+F 0 "FID3" H 3435 1946 50  0000 L CNN
+F 1 "Fiducial" H 3435 1855 50  0000 L CNN
+F 2 "Fiducial:Fiducial_0.75mm_Mask1.5mm" H 3350 1900 50  0001 C CNN
+F 3 "~" H 3350 1900 50  0001 C CNN
+	1    3350 1900
+	1    0    0    -1
+$EndComp
 $EndSCHEMATC

Commit message: add digikey part number
Parts:
- D2: PRICE (none) -> 0.68; digikey# (none) -> 350-4358-2-ND
- D3: PRICE (none) -> 0.065; digikey# (none) -> 3372-0805RBD0070S01TR-ND
- J1: PRICE (none) -> 0.33; digikey# (none) -> 2057-MCR-B-S-RA-TSMT-NP-CS4-T/R-ND
- J2: PRICE 0.71 USD -> 0.62; digikey# (none) -> CONUFL001-SMD-TTR-ND
- J3: PRICE (none) -> 9.97; digikey# (none) -> 732-13840-ND
- J4: PRICE (none) -> 0.66; digikey (none) -> 2073-BC020-03-A-0200-0300-L-G-ND
- J5: PRICE (none) -> 0.14; digikey (none) -> 664-G800LF306018EU-ND
- J6: PRICE (none) -> 0.14; digikey# (none) -> 664-G800LF306018EU-ND
- J7: PRICE (none) -> 0.66; digikey# (none) -> 2073-BC020-03-A-0200-0300-L-G-ND
- U2: PRICE (none) -> 1.13; digikey# (none) -> MCP6021RT-E/OTTR-ND
- U3: PRICE (none) -> 0.55; digikey# (none) -> 497-6447-2-ND
- U4: PRICE (none) -> 13.44; digikey# (none) -> RFM95W-915S2-ND
- U5: PRICE (none) -> 9.34; digikey# (none) -> ESP-12SRF-ND
Connections:
- wire segments 111 -> 112
Changed lines of the file:
@@
 F 2 "Package_TO_SOT_SMD:SOT-223-3_TabPin2" H 4000 6300 50  0001 C CNN
 F 3 "http://www.st.com/st-web-ui/static/active/en/resource/technical/document/datasheet/CD00000544.pdf" H 4100 5850 50  0001 C CNN
+F 4 "497-6447-2-ND" H 4000 6100 50  0001 C CNN "digikey#"
+F 5 "0.55" H 4000 6100 50  0001 C CNN "PRICE"
 	1    4000 6100
 	1    0    0    -1
@@
 Wire Wire Line
 	4300 6100 4600 6100
-Wire Wire Line
-	4600 6100 4600 5700
 Connection ~ 4600 6100
 Wire Wire Line
@@
 F 2 "RFUFL2:HRS_U.FL-R-SMT-1(10)" H 6350 1550 50  0001 L BNN
 F 3 "https://www.farnell.com/datasheets/2691132.pdf" H 6350 1550 50  0001 L BNN
-F 4 "0.71 USD" H 6350 1550 50  0001 L BNN "PRICE"
+F 4 "0.62" H 6350 1550 50  0001 L BNN "PRICE"
 F 5 "None" H 6350 1550 50  0001 L BNN "PACKAGE"
 F 6 "Manufacturer Recommendation" H 6350 1550 50  0001 L BNN "STANDARD"
@@
 F 9 "Hirose" H 6350 1550 50  0001 L BNN "MANUFACTURER"
 F 10 "Good" H 6350 1550 50  0001 L BNN "AVAILABILITY"
+F 11 "CONUFL001-SMD-TTR-ND" H 6350 1550 50  0001 C CNN "digikey#"
 	1    6350 1550
 	-1   0    0    -1
@@
 F 5 "AMPHENOL CONEXX" H 7800 1650 50  0001 L BNN "MANUFACTURER"
 F 6 "C" H 7800 1650 50  0001 L BNN "PARTREV"
+F 7 "732-13840-ND" H 7800 1650 50  0001 C CNN "digikey#"
+F 8 "9.97" H 7800 1650 50  0001 C CNN "PRICE"
 	1    7800 1650
 	1    0    0    -1
@@
 F 2 "RF_Module:HOPERF_RFM9XW_SMD" H 3550 5200 50  0001 C CNN
 F 3 "https://www.hoperf.com/data/upload/portal/20181127/5bfcbea20e9ef.pdf" H 3550 5200 50  0001 C CNN
+F 4 "RFM95W-915S2-ND" H 6850 3550 50  0001 C CNN "digikey#"
+F 5 "13.44" H 6850 3550 50  0001 C CNN "PRICE"
 	1    6850 3550
 	-1   0    0    1
@@
 F 2 "Connector_PinHeader_2.54mm:PinHeader_1x03_P2.54mm_Vertical" H 10250 2700 50  0001 C CNN
 F 3 "~" H 10250 2700 50  0001 C CNN
+F 4 "2073-BC020-03-A-0200-0300-L-G-ND" H 10250 2700 50  0001 C CNN "digikey"
+F 5 "0.66" H 10250 2700 50  0001 C CNN "PRICE"
 	1    10250 2700
 	1    0    0    -1
@@
 F 2 "Connector_PinHeader_2.54mm:PinHeader_1x02_P2.54mm_Vertical" H 10250 3800 50  0001 C CNN
 F 3 "~" H 10250 3800 50  0001 C CNN
+F 4 "664-G800LF306018EU-ND" H 10250 3800 50  0001 C CNN "digikey"
+F 5 "0.14" H 10250 3800 50  0001 C CNN "PRICE"
 	1    10250 3800
 	1    0    0    -1
@@
 F 2 "LED_SMD:LED_0805_2012Metric_Castellated" H 8200 5150 50  0001 C CNN
 F 3 "~" H 8200 5150 50  0001 C CNN
+F 4 "3372-0805RBD0070S01TR-ND" V 8200 5150 50  0001 C CNN "digikey#"
+F 5 "0.065" V 8200 5150 50  0001 C CNN "PRICE"
 	1    8200 5150
 	0    -1   -1   0
@@
 F 2 "LED_SMD:LED_0805_2012Metric_Castellated" H 7900 5150 50  0001 C CNN
 F 3 "~" H 7900 5150 50  0001 C CNN
+F 4 "350-4358-2-ND" V 7900 5150 50  0001 C CNN "digikey#"
+F 5 "0.68" V 7900 5150 50  0001 C CNN "PRICE"
 	1    7900 5150
 	0    -1   -1   0
@@
 F 2 "Connector_PinHeader_2.54mm:PinHeader_1x02_P2.54mm_Vertical" H 10250 4500 50  0001 C CNN
 F 3 "~" H 10250 4500 50  0001 C CNN
+F 4 "664-G800LF306018EU-ND" H 10250 4500 50  0001 C CNN "digikey#"
+F 5 "0.14" H 10250 4500 50  0001 C CNN "PRICE"
 	1    10250 4500
 	1    0    0    -1
@@
 F 2 "Connector_USB:USB_Mini-B_Lumberg_2486_01_Horizontal" H 2000 6250 50  0001 C CNN
 F 3 "https://www.farnell.com/datasheets/2347419.pdf" H 2000 6250 50  0001 C CNN
+F 4 "2057-MCR-B-S-RA-TSMT-NP-CS4-T/R-ND " H 1850 6300 50  0001 C CNN "digikey#"
+F 5 "0.33" H 1850 6300 50  0001 C CNN "PRICE"
 	1    1850 6300
 	1    0    0    -1
@@
 L power:PWR_FLAG #FLG0102
 U 1 1 60E3DDB4
-P 5000 6850
-F 0 "#FLG0102" H 5000 6925 50  0001 C CNN
-F 1 "PWR_FLAG" H 5000 7023 50  0000 C CNN
-F 2 "" H 5000 6850 50  0001 C CNN
-F 3 "~" H 5000 6850 50  0001 C CNN
-	1    5000 6850
-	1    0    0    -1
-$EndComp
-$Comp
-L power:GND #PWR0105
-U 1 1 60E3E607
-P 5000 7050
-F 0 "#PWR0105" H 5000 6800 50  0001 C CNN
-F 1 "GND" H 5005 6877 50  0000 C CNN
-F 2 "" H 5000 7050 50  0001 C CNN
-F 3 "" H 5000 7050 50  0001 C CNN
-	1    5000 7050
-	1    0    0    -1
-$EndComp
-Wire Wire Line
-	5000 6850 5000 7050
+P 2300 7100
+F 0 "#FLG0102" H 2300 7175 50  0001 C CNN
+F 1 "PWR_FLAG" H 2300 7273 50  0000 C CNN
+F 2 "" H 2300 7100 50  0001 C CNN
+F 3 "~" H 2300 7100 50  0001 C CNN
+	1    2300 7100
+	-1   0    0    1
+$EndComp
 Wire Wire Line
 	6450 1550 7000 1550
@@
 F 3 "http://ww1.microchip.com/downloads/en/devicedoc/20001685e.pdf" H 3650 3800 50  0001 L BNN
 F 4 "IC-12504" H 3650 3800 50  0001 L BNN "PROD_ID"
+F 5 "MCP6021RT-E/OTTR-ND" H 3650 3800 50  0001 C CNN "digikey#"
+F 6 "1.13" H 3650 3800 50  0001 C CNN "PRICE"
 	1    3650 3800
 	1    0    0    -1
@@
 F 3 "https://docs.ai-thinker.com/_media/esp8266/docs/esp-12s_product_specification_en.pdf" H 8650 3650 50  0001 L BNN
 F 4 "IC-14115" H 8650 3650 50  0001 L BNN "PROD_ID"
+F 5 "ESP-12SRF-ND" H 8650 3650 50  0001 C CNN "digikey#"
+F 6 "9.34" H 8650 3650 50  0001 C CNN "PRICE"
 	1    8650 3650
 	-1   0    0    -1
@@
 F 2 "Connector_PinHeader_2.54mm:PinHeader_1x03_P2.54mm_Vertical" H 1800 3900 50  0001 C CNN
 F 3 "~" H 1800 3900 50  0001 C CNN
+F 4 "2073-BC020-03-A-0200-0300-L-G-ND" H 1800 3900 50  0001 C CNN "digikey#"
+F 5 "0.66" H 1800 3900 50  0001 C CNN "PRICE"
 	1    1800 3900
 	-1   0    0    1
@@
 	1    0    0    -1
 $EndComp
+Wire Wire Line
+	4600 5700 4600 6100
+Wire Wire Line
+	2300 7100 2300 6800
+Wire Wire Line
+	2300 6800 1850 6800
 $EndSCHEMATC

Commit message: add ruteo
Other:
- note added: "MIcrocontrolador y radio LoRa"
- moved on the sheet: C1, C2, C3, C4, C5, C6, C7, D1, D2, D3, FID1, FID2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

Commit message: correcciones revisiones del docente
Other:
- note added: "Línea de transmisión \ntipo coplanar con plano de tierra\nImpedancia 50 ohm\nAncho de pista 0,3 mm\n"
Changed lines of the file:
@@
 Wire Notes Line
 	8200 1950 8700 1950
+Text Notes 7500 2950 0    50   ~ 0
+Línea de transmisión \ntipo coplanar con plano de tierra\nImpedancia 50 ohm\nAncho de pista 0,3 mm\n
+Wire Notes Line
+	7050 2900 7200 2800
+Wire Notes Line
+	7200 2800 7450 2800
 $EndSCHEMATC
